Commit message: Update urdf file

File: urdf/hachibot.urdf (robot description, URDF)
Before this commit: robot hachibot, 5 links, 4 joints
Links:
- link left_back_wheel: geometry visual cylinder length=0.06 radius=0.065
- link left_front_wheel: geometry visual cylinder length=0.06 radius=0.065
- link right_back_wheel: geometry visual cylinder length=0.06 radius=0.065
- link right_front_wheel: geometry visual cylinder length=0.06 radius=0.065
